File: knipper.sch (KiCad schematic (older format))
At the start: 30 parts, among them J1 INPUT, J2 5V_REV_FROM_CONTROLLER, J3 REVLIGHTS, J4 DIR_RIGHT, J5 DIR_LEFT, Q1 IRF520N, Q2 IRF520N, Q3 IRF520N, SW5 DIRECTION_SWITCH, U1 NE555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

Commit message: implemented high side switching
Parts:
- removed C1: 10uF, Capacitors_THT:CP_Radial_D5.0mm_P2.50mm, symbol C
- removed H5, H6: MOUNT_HOLE, knipper:MountingHole_3mm, symbol MOUNT_HOLE
- removed Q1, Q2, Q3: IRF520N, TO_SOT_Packages_THT:TO-220_Vertical, symbol IRF540N
- added C1: 10uF, Capacitors_THT:CP_Radial_D5.0mm_P2.50mm, symbol CP
- added Q1, Q2, Q3: 2N3904, TO_SOT_Packages_THT:TO-92_Molded_Narrow, symbol 2N3904
- added Q4, Q5, Q6: IRF5210PBF, TO_SOT_Packages_THT:TO-220-3_Vertical, symbol IRF5210PBF
- added R10: 47k, Resistors_THT:R_Axial_DIN0207_L6.3mm_D2.5mm_P7.62mm_Horizontal, symbol R
- added R11, R12, R13: 4k7, Resistors_THT:R_Axial_DIN0207_L6.3mm_D2.5mm_P7.62mm_Horizontal, symbol R
- C2: footprint Capacitors_THT:C_Axial_L5.1mm_D3.1mm_P7.50mm_Horizontal -> Capacitors_THT:C_Disc_D5.0mm_W2.5mm_P5.00mm
- J3: value REVLIGHTS -> REVLIGHT
- R6, R7: value 1k -> 47k
- R9: value 1k -> 10k
Connections:
- net +12V: now also Q4.3 (S), Q5.3 (S), Q6.3 (S), R11.2, R12.2, R13.2
- net DIR_L: now also Q4.2 (D)
- net DIR_R: now also Q5.2 (D)
- net GND: now also R9.1, C1.2, Q1.1 (E), Q2.1 (E), Q3.1 (E); no longer J2.1 (Pin_1), U4.2
- net at R2.2, U1.2 (TR), U1.6 (THR): now also C1.1
- net at R7.1: now also Q2.2 (B)
- net at R6.1: now also Q1.2 (B)
- net at J3.1 (Pin_1): now also Q6.2 (D)
- net at R9.2, U4.3: now also R10.2
- new net: Q1.3 (C), Q4.1 (G), R11.1
- new net: Q2.3 (C), Q5.1 (G), R12.1
- new net: Q3.3 (C), Q6.1 (G), R13.1
- new net: Q3.2 (B), R10.1
- new net E-GND: J2.1 (Pin_1), U4.2
Other:
- moved on the sheet: J3, J4, J5, R7

Commit message: Changed parts and layout to SMD
Parts:
- removed Q6: IRF5210PBF, TO_SOT_Packages_THT:TO-220-3_Vertical, symbol IRF5210PBF
- removed R2: 50K, Resistors_THT:R_Axial_DIN0207_L6.3mm_D2.5mm_P7.62mm_Horizontal, symbol R_Variable
- added Q4: IRF5210STRLPBF, TO_SOT_Packages_SMD:TO-263-3_TabPin2, symbol IRF5210PBF
- added R2: 100K, Potentiometers:Potentiometer_Trimmer_Vishay_TS53YJ, symbol POT
- C1: footprint Capacitors_THT:CP_Radial_D5.0mm_P2.50mm -> Capacitors_SMD:C_1206_HandSoldering; Farnell (none) -> 1457413
- C2: footprint Capacitors_THT:C_Disc_D5.0mm_W2.5mm_P5.00mm -> Capacitors_SMD:C_0603_HandSoldering; Farnell (none) -> 1414609
- Q1, Q2, Q3: value 2N3904 -> BSR14; footprint TO_SOT_Packages_THT:TO-92_Molded_Narrow -> TO_SOT_Packages_SMD:SOT-23; Farnell (none) -> 1700688
- Q5: value IRF5210PBF -> IRF5210STRLPBF; footprint TO_SOT_Packages_THT:TO-220-3_Vertical -> TO_SOT_Packages_SMD:TO-263-3_TabPin2; Farnell (none) -> 1298529
- Q6: renamed from Q4; value IRF5210PBF -> IRF5210STRLPBF; footprint TO_SOT_Packages_THT:TO-220-3_Vertical -> TO_SOT_Packages_SMD:TO-263-3_TabPin2; Farnell (none) -> 1298529
- R1, R10, R11, R12, R13, R3, R4, R5, R6, R7, R9: footprint Resistors_THT:R_Axial_DIN0207_L6.3mm_D2.5mm_P7.62mm_Horizontal -> Resistors_SMD:R_0603_HandSoldering
- R8: footprint Resistors_THT:R_Axial_DIN0207_L6.3mm_D2.5mm_P7.62mm_Horizontal -> Resistors_SMD:R_0805_HandSoldering
- U1: value NE555 -> NE555D; footprint Housings_DIP:DIP-8_W7.62mm -> Housings_SOIC:SOIC-8_3.9x4.9mm_Pitch1.27mm; Farnell (none) -> 2782865
- U2: value 4071 -> CD4071BM; footprint Housings_DIP:DIP-14_W7.62mm_LongPads -> SMD_Packages:SOIC-14_N; Farnell (none) -> 1739909
- U3: value 4081 -> CD4081BM; footprint Housings_DIP:DIP-14_W7.62mm_LongPads -> SMD_Packages:SOIC-14_N; Farnell (none) -> 1122563
- U4: value LTV-814 -> FOD814SD; footprint Housings_DIP:DIP-4_W7.62mm -> Housings_DIP:SMDIP-4_W9.53mm; Farnell (none) -> 2453194
Connections:
- net +12V: now also Q4.3 (S)
- net DIR_L: now also Q4.2 (D); no longer Q6.2 (D)
- net at C1.1, U1.2 (TR), U1.6 (THR): now also R2.2, R2.3
- net at R1.2, U1.7 (DIS): now also R2.1
- net at J3.1 (Pin_1): now also Q6.2 (D)
- net at Q1.3 (C), R11.1: now also Q4.1 (G); no longer Q6.1 (G)
- net at Q3.3 (C), R13.1: now also Q6.1 (G)
Other:
- moved on the sheet: Q6
